Commit message: fix: Di chuyển pusher_controllers.yaml sang sorting_robot_controller và stagger spawn controller để khắc phục lỗi load controller
- Chuyển file pusher_controllers.yaml từ sorting_robot_description sang sorting_robot_controller để tránh controller_manager corrupt tham số --params-file khi đường dẫn chứa chuỗi "robot_description"
- Thêm RegisterEventHandler, TimerAction và OnProcessExit để spawn joint_state_broadcaster sau 6 giây khi spawn_pusher exit, rồi spawn pusher_position_controller sau khi joint_state_broadcaster exit
- Thêm --controller-manager-timeout 60 cho các spawner node
- Cập nhật controllers_config trong pusher.launch.py trỏ sang package sorting_robot_controller
- Thêm exec_depend sorting_robot_controller trong package.xml
- Xóa cài đặt thư mục config khỏi setup.py
- Điều chỉnh base_y, base_z và stroke của pusher trong pusher.urdf.xacro

File: src/sorting_robot_description/urdf/pusher.urdf.xacro (robot description, xacro)
@@ -9,8 +9,8 @@
   <!-- Pose of the pusher base in the world (beside the belt end). -->
   <xacro:property name="base_x" value="0.6"/>
-  <xacro:property name="base_y" value="0.5"/>
-  <xacro:property name="base_z" value="0.575"/>
+  <xacro:property name="base_y" value="0.35"/>
+  <xacro:property name="base_z" value="0.615"/>
   <!-- Prismatic stroke (m): 0 = retracted (clear of belt), negative = across. -->
-  <xacro:property name="stroke" value="0.85"/>
+  <xacro:property name="stroke" value="0.70"/>
   <material name="pusher_orange">
     <color rgba="0.9 0.45 0.1 1"/>

Commit message: feat: Tích hợp toàn bộ pipeline phân loại qua `system.launch.py` và cải thiện timing đẩy cube
* Thêm `system.launch.py` khởi chạy Gazebo, vision, decision, pusher và spawner với stagger startup
* Thêm `system_params.yaml` tập trung tham số của toàn bộ các node
* Di chuyển camera trong `conveyor.world` lên trên pusher (x=0.6) để phát hiện cube ngay tại paddle
* Thêm ROI detection trong `vision_node` giới hạn vùng phát hiện quanh pusher
* Thêm position gate trong `decision_node` kích hoạt reject theo vị trí centroid thay vì thời gian
* Sửa rò rỉ timer trong `pusher_controller_node` bằng cách destroy timer thay vì chỉ cancel
* Tăng effort/velocity và giảm damping/friction của pusher joint trong `pusher.urdf.xacro`

File: src/sorting_robot_description/urdf/pusher.urdf.xacro (robot description, xacro)
@@ -48,6 +48,10 @@
     <origin xyz="0 0 0" rpy="0 0 0"/>
     <axis xyz="0 1 0"/>
-    <limit lower="-${stroke}" upper="0.0" effort="50.0" velocity="1.5"/>
-    <dynamics damping="1.0" friction="0.5"/>
+    <!-- High effort + speed so the belt-driven cube's resistance is negligible
+         and the stroke always completes within the fixed extend_time, keeping
+         the push timing deterministic for the cubes queued behind. Low
+         damping/friction so the joint is not sluggish. -->
+    <limit lower="-${stroke}" upper="0.0" effort="300.0" velocity="3.0"/>
+    <dynamics damping="0.05" friction="0.0"/>
   </joint>
   <!-- Paddle that contacts the cube. -->
