Commit message: feat(bringup): Tích hợp myCobot 280 với Gazebo Sim và ros2_control cho demo pick-and-place
* Thêm `bringup.launch.py` để khởi động Gazebo Sim, spawn robot, bridge `/clock` và stagger controller spawner
* Thêm `controllers.yaml` cấu hình `joint_state_broadcaster`, `arm_controller` và `gripper_controller`
* Thêm `pick_world.sdf` với mặt bàn và physics step 4ms để tối ưu RTF
* Thêm `ros_gz_bridge.yaml` cho topic `/clock`
* Đổi tên khớp gripper từ `gripper_controller` sang `gripper_finger_joint` để tránh xung đột tên controller
* Thay thế collision mesh bằng box primitive trên arm và gripper để giảm tải physics
* Thêm tham số `mount_z` vào URDF để đặt độ cao base robot
* Cập nhật `Makefile` với target `gz`, `gz-test`, `view`, `check` và `kill`
* Cập nhật `package.xml` và `CMakeLists.txt` để cài đặt config, worlds và dependencies mới

File: src/mycobot_description/urdf/mycobot_280.ros2_control.xacro (robot description, xacro)
@@ -24,5 +24,5 @@
       <xacro:arm_joint jname="joint6_to_joint5"/>
       <xacro:arm_joint jname="joint6output_to_joint6"/>
-      <joint name="gripper_controller">
+      <joint name="gripper_finger_joint">
         <command_interface name="position"/>
         <state_interface name="position"/>

File: src/mycobot_description/urdf/mycobot_280.urdf.xacro (robot description, xacro)
@@ -11,4 +11,5 @@
   <xacro:arg name="use_gz" default="true"/>
   <xacro:arg name="use_world_fixed" default="true"/>
+  <xacro:arg name="mount_z" default="0.0"/>
   <xacro:arg name="controllers_config" default=""/>
   <xacro:include filename="$(find mycobot_description)/urdf/inertials.xacro"/>
@@ -18,8 +19,11 @@
   <xacro:if value="$(arg use_world_fixed)">
     <link name="world"/>
+    <!-- mount_z: chiều cao đặt base so với world (mặt bàn ở 0.4 khi chạy Gazebo).
+         Đặt độ cao ngay tại đây thay vì offset lúc spawn, vì gz ghim link `world`
+         vào gốc thế giới và bỏ qua -z lúc spawn. -->
     <joint name="world_to_g_base" type="fixed">
       <parent link="world"/>
       <child link="g_base"/>
-      <origin xyz="0 0 0" rpy="0 0 0"/>
+      <origin xyz="0 0 $(arg mount_z)" rpy="0 0 0"/>
     </joint>
   </xacro:if>

File: src/mycobot_description/urdf/mycobot_280_arm.xacro (robot description, xacro)
@@ -18,6 +18,6 @@
     </visual>
     <collision>
-      <geometry><mesh filename="${mesh}/G_base.dae"/></geometry>
-      <origin xyz="0.0 0 -0.032" rpy="0 0 1.5708"/>
+      <geometry><box size="0.09 0.09 0.06"/></geometry>
+      <origin xyz="0 0 -0.02" rpy="0 0 0"/>
     </collision>
     <xacro:box_inertial mass="0.5" size="0.05"/>
@@ -29,6 +29,6 @@
     </visual>
     <collision>
-      <geometry><mesh filename="${mesh}/joint1.dae"/></geometry>
-      <origin xyz="0 0 0" rpy="0 0 -3.14159"/>
+      <geometry><box size="0.08 0.08 0.09"/></geometry>
+      <origin xyz="0 0 0.06" rpy="0 0 0"/>
     </collision>
     <xacro:box_inertial mass="0.3" size="0.04"/>
@@ -40,6 +40,6 @@
     </visual>
     <collision>
-      <geometry><mesh filename="${mesh}/joint2.dae"/></geometry>
-      <origin xyz="0 0 -0.06096" rpy="0 0 -1.5708"/>
+      <geometry><box size="0.06 0.06 0.08"/></geometry>
+      <origin xyz="0 0 -0.03" rpy="0 0 0"/>
     </collision>
     <xacro:box_inertial mass="0.3" size="0.04"/>
@@ -51,6 +51,6 @@
     </visual>
     <collision>
-      <geometry><mesh filename="${mesh}/joint3.dae"/></geometry>
-      <origin xyz="0 0 0.03256" rpy="0 -1.5708 0"/>
+      <geometry><box size="0.09 0.06 0.06"/></geometry>
+      <origin xyz="-0.05 0 0.03" rpy="0 0 0"/>
     </collision>
     <xacro:box_inertial mass="0.25" size="0.04"/>
@@ -62,6 +62,6 @@
     </visual>
     <collision>
-      <geometry><mesh filename="${mesh}/joint4.dae"/></geometry>
-      <origin xyz="0 0 0.03056" rpy="0 -1.5708 0"/>
+      <geometry><box size="0.08 0.06 0.06"/></geometry>
+      <origin xyz="-0.04 0 0.03" rpy="0 0 0"/>
     </collision>
     <xacro:box_inertial mass="0.2" size="0.035"/>
@@ -73,6 +73,6 @@
     </visual>
     <collision>
-      <geometry><mesh filename="${mesh}/joint5.dae"/></geometry>
-      <origin xyz="0 0 -0.03356" rpy="-1.5708 0 0"/>
+      <geometry><box size="0.05 0.06 0.05"/></geometry>
+      <origin xyz="0 0 -0.03" rpy="0 0 0"/>
     </collision>
     <xacro:box_inertial mass="0.2" size="0.035"/>
@@ -84,6 +84,6 @@
     </visual>
     <collision>
-      <geometry><mesh filename="${mesh}/joint6.dae"/></geometry>
-      <origin xyz="0 0 -0.038" rpy="0 0 0"/>
+      <geometry><box size="0.045 0.045 0.03"/></geometry>
+      <origin xyz="0 0 -0.02" rpy="0 0 0"/>
     </collision>
     <xacro:box_inertial mass="0.15" size="0.03"/>
@@ -95,6 +95,6 @@
     </visual>
     <collision>
-      <geometry><mesh filename="${mesh}/joint7.dae"/></geometry>
-      <origin xyz="0 0 -0.012" rpy="0 0 0"/>
+      <geometry><box size="0.04 0.04 0.02"/></geometry>
+      <origin xyz="0 0 -0.01" rpy="0 0 0"/>
     </collision>
     <xacro:box_inertial mass="0.1" size="0.02"/>

File: src/mycobot_description/urdf/mycobot_280_gripper.xacro (robot description, xacro)
@@ -3,12 +3,29 @@
   <!--
     Gripper thích ứng (adaptive) của myCobot 280.
-    Chỉ 1 khớp thật `gripper_controller` được điều khiển; 5 khớp còn lại `mimic`
-    theo nó (đóng/mở đồng bộ) - đã có sẵn trong URDF gốc của Elephant Robotics.
-    Đã thêm inertial + velocity limit dương. Thêm frame `grasp_center` làm điểm
-    gắp (attach vật + MoveIt end-effector).
+    - Chỉ 1 khớp thật `gripper_finger_joint` được điều khiển; 5 khớp còn lại `mimic`.
+      (Đổi tên khớp gốc `gripper_controller` -> `gripper_finger_joint` để KHÔNG trùng
+       tên controller `gripper_controller`, tránh lỗi controller_manager tưởng là
+       reference interface của controller chainable.)
+    - Collision dùng box primitive (không phải mesh) để nhẹ physics, tăng RTF.
+    - `grasp_center`: điểm gắp (attach vật + MoveIt end-effector).
+    - LƯU Ý: physics engine của Gazebo không ràng buộc <mimic> (chỉ cảnh báo, non-fatal);
+      với grasp attach/detach thì không ảnh hưởng.
   -->
   <xacro:property name="gmesh" value="package://mycobot_description/meshes/adaptive_gripper"/>
   <xacro:property name="gvel" value="2.0"/>
   <xacro:property name="geff" value="20.0"/>
+  <xacro:macro name="finger_link" params="name mesh_file ox oy oz">
+    <link name="${name}">
+      <visual>
+        <geometry><mesh filename="${gmesh}/${mesh_file}"/></geometry>
+        <origin xyz="${ox} ${oy} ${oz}" rpy="0 0 0"/>
+      </visual>
+      <collision>
+        <geometry><box size="0.02 0.03 0.01"/></geometry>
+        <origin xyz="${ox} ${oy} ${oz}" rpy="0 0 0"/>
+      </collision>
+      <xacro:box_inertial mass="0.02" size="0.015"/>
+    </link>
+  </xacro:macro>
   <!-- Nối gripper vào flange của cánh tay -->
   <joint name="joint6output_to_gripper_base" type="fixed">
@@ -23,53 +40,17 @@
     </visual>
     <collision>
-      <geometry><mesh filename="${gmesh}/gripper_base.dae"/></geometry>
+      <geometry><box size="0.05 0.03 0.03"/></geometry>
       <origin xyz="0 0 -0.012" rpy="0 0 0"/>
     </collision>
     <xacro:box_inertial mass="0.1" size="0.03"/>
   </link>
-  <link name="gripper_left1">
-    <visual><geometry><mesh filename="${gmesh}/gripper_left1.dae"/></geometry>
-      <origin xyz="0.039 -0.0133 -0.012" rpy="0 0 0"/></visual>
-    <collision><geometry><mesh filename="${gmesh}/gripper_left1.dae"/></geometry>
-      <origin xyz="0.039 -0.0133 -0.012" rpy="0 0 0"/></collision>
-    <xacro:box_inertial mass="0.02" size="0.015"/>
-  </link>
-  <link name="gripper_left2">
-    <visual><geometry><mesh filename="${gmesh}/gripper_left2.dae"/></geometry>
-      <origin xyz="0.005 -0.0195 -0.012" rpy="0 0 0"/></visual>
-    <collision><geometry><mesh filename="${gmesh}/gripper_left2.dae"/></geometry>
-      <origin xyz="0.005 -0.0195 -0.012" rpy="0 0 0"/></collision>
-    <xacro:box_inertial mass="0.02" size="0.015"/>
-  </link>
-  <link name="gripper_left3">
-    <visual><geometry><mesh filename="${gmesh}/gripper_left3.dae"/></geometry>
-      <origin xyz="0.012 0.0025 -0.012" rpy="0 0 0"/></visual>
-    <collision><geometry><mesh filename="${gmesh}/gripper_left3.dae"/></geometry>
-      <origin xyz="0.012 0.0025 -0.012" rpy="0 0 0"/></collision>
-    <xacro:box_inertial mass="0.02" size="0.015"/>
-  </link>
-  <link name="gripper_right1">
-    <visual><geometry><mesh filename="${gmesh}/gripper_right1.dae"/></geometry>
-      <origin xyz="-0.039 -0.0133 -0.012" rpy="0 0 0"/></visual>
-    <collision><geometry><mesh filename="${gmesh}/gripper_right1.dae"/></geometry>
-      <origin xyz="-0.039 -0.0133 -0.012" rpy="0 0 0"/></collision>
-    <xacro:box_inertial mass="0.02" size="0.015"/>
-  </link>
-  <link name="gripper_right2">
-    <visual><geometry><mesh filename="${gmesh}/gripper_right2.dae"/></geometry>
-      <origin xyz="-0.005 -0.0195 -0.012" rpy="0 0 0"/></visual>
-    <collision><geometry><mesh filename="${gmesh}/gripper_right2.dae"/></geometry>
-      <origin xyz="-0.005 -0.0195 -0.012" rpy="0 0 0"/></collision>
-    <xacro:box_inertial mass="0.02" size="0.015"/>
-  </link>
-  <link name="gripper_right3">
-    <visual><geometry><mesh filename="${gmesh}/gripper_right3.dae"/></geometry>
-      <origin xyz="-0.012 0.0025 -0.012" rpy="0 0 0"/></visual>
-    <collision><geometry><mesh filename="${gmesh}/gripper_right3.dae"/></geometry>
-      <origin xyz="-0.012 0.0025 -0.012" rpy="0 0 0"/></collision>
-    <xacro:box_inertial mass="0.02" size="0.015"/>
-  </link>
-  <!-- Khớp điều khiển chính -->
-  <joint name="gripper_controller" type="revolute">
+  <xacro:finger_link name="gripper_left1"  mesh_file="gripper_left1.dae"  ox="0.039"  oy="-0.0133" oz="-0.012"/>
+  <xacro:finger_link name="gripper_left2"  mesh_file="gripper_left2.dae"  ox="0.005"  oy="-0.0195" oz="-0.012"/>
+  <xacro:finger_link name="gripper_left3"  mesh_file="gripper_left3.dae"  ox="0.012"  oy="0.0025"  oz="-0.012"/>
+  <xacro:finger_link name="gripper_right1" mesh_file="gripper_right1.dae" ox="-0.039" oy="-0.0133" oz="-0.012"/>
+  <xacro:finger_link name="gripper_right2" mesh_file="gripper_right2.dae" ox="-0.005" oy="-0.0195" oz="-0.012"/>
+  <xacro:finger_link name="gripper_right3" mesh_file="gripper_right3.dae" ox="-0.012" oy="0.0025"  oz="-0.012"/>
+  <!-- Khớp điều khiển chính (đã đổi tên) -->
+  <joint name="gripper_finger_joint" type="revolute">
     <axis xyz="0 0 1"/>
     <limit effort="${geff}" lower="-0.74" upper="0.15" velocity="${gvel}"/>
@@ -84,5 +65,5 @@
     <child link="gripper_left2"/>
     <origin xyz="-0.005 0.027 0" rpy="0 0 0"/>
-    <mimic joint="gripper_controller" multiplier="1.0" offset="0"/>
+    <mimic joint="gripper_finger_joint" multiplier="1.0" offset="0"/>
   </joint>
   <joint name="gripper_left3_to_gripper_left1" type="revolute">
@@ -92,5 +73,5 @@
     <child link="gripper_left1"/>
     <origin xyz="-0.027 0.016 0" rpy="0 0 0"/>
-    <mimic joint="gripper_controller" multiplier="-1.0" offset="0"/>
+    <mimic joint="gripper_finger_joint" multiplier="-1.0" offset="0"/>
   </joint>
   <joint name="gripper_base_to_gripper_right3" type="revolute">
@@ -100,5 +81,5 @@
     <child link="gripper_right3"/>
     <origin xyz="0.012 0.005 0" rpy="0 0 0"/>
-    <mimic joint="gripper_controller" multiplier="-1.0" offset="0"/>
+    <mimic joint="gripper_finger_joint" multiplier="-1.0" offset="0"/>
   </joint>
   <joint name="gripper_base_to_gripper_right2" type="revolute">
@@ -108,5 +89,5 @@
     <child link="gripper_right2"/>
     <origin xyz="0.005 0.027 0" rpy="0 0 0"/>
-    <mimic joint="gripper_controller" multiplier="-1.0" offset="0"/>
+    <mimic joint="gripper_finger_joint" multiplier="-1.0" offset="0"/>
   </joint>
   <joint name="gripper_right3_to_gripper_right1" type="revolute">
@@ -116,8 +97,7 @@
     <child link="gripper_right1"/>
     <origin xyz="0.027 0.016 0" rpy="0 0 0"/>
-    <mimic joint="gripper_controller" multiplier="1.0" offset="0"/>
+    <mimic joint="gripper_finger_joint" multiplier="1.0" offset="0"/>
   </joint>
-  <!-- Điểm gắp: nằm giữa 2 ngón, dùng cho attach vật + MoveIt EE.
-       Offset tạm; sẽ tinh chỉnh khi xem trong RViz/Gazebo (Phase 6/7). -->
+  <!-- Điểm gắp: giữa 2 ngón, dùng cho attach vật + MoveIt EE. Offset tạm, tinh chỉnh Phase 6/7. -->
   <link name="grasp_center"/>
   <joint name="gripper_base_to_grasp_center" type="fixed">

Commit message: feat: Thêm package `mycobot_demo` và sửa gripper URDF cho Phase 3
* Thêm package `mycobot_demo` với node `test_arm` và `test_gripper` để kiểm tra trajectory và gripper
* Thêm target `test-arm` và `test-gripper` vào Makefile
* Thêm `gripper_right_joint` vào `controllers.yaml` và `mycobot_280.ros2_control.xacro`
* Sửa gripper URDF: bỏ khớp `mimic`, chuyển sang 2 khớp điều khiển đối xứng (`gripper_finger_joint` và `gripper_right_joint`)
* Bỏ collision geometry cho các link ngón gripper để tránh kẹt vật lý

File: src/mycobot_description/urdf/mycobot_280.ros2_control.xacro (robot description, xacro)
@@ -29,4 +29,9 @@
         <state_interface name="velocity"/>
       </joint>
+      <joint name="gripper_right_joint">
+        <command_interface name="position"/>
+        <state_interface name="position"/>
+        <state_interface name="velocity"/>
+      </joint>
     </ros2_control>
   </xacro:macro>

File: src/mycobot_description/urdf/mycobot_280_gripper.xacro (robot description, xacro)
@@ -2,17 +2,18 @@
 <robot xmlns:xacro="http://www.ros.org/wiki/xacro">
   <!--
-    Gripper thích ứng (adaptive) của myCobot 280.
-    - Chỉ 1 khớp thật `gripper_finger_joint` được điều khiển; 5 khớp còn lại `mimic`.
-      (Đổi tên khớp gốc `gripper_controller` -> `gripper_finger_joint` để KHÔNG trùng
-       tên controller `gripper_controller`, tránh lỗi controller_manager tưởng là
-       reference interface của controller chainable.)
-    - Collision dùng box primitive (không phải mesh) để nhẹ physics, tăng RTF.
-    - `grasp_center`: điểm gắp (attach vật + MoveIt end-effector).
-    - LƯU Ý: physics engine của Gazebo không ràng buộc <mimic> (chỉ cảnh báo, non-fatal);
-      với grasp attach/detach thì không ảnh hưởng.
+    Gripper myCobot 280 (bản đơn giản hoá cho Gazebo).
+    - Hai khớp gốc ngón được ĐIỀU KHIỂN đối xứng:
+        gripper_finger_joint  (ngón trái, gripper_left3)   : đóng khi ÂM
+        gripper_right_joint   (ngón phải, gripper_right3)  : đóng khi DƯƠNG (đối xứng)
+    - Bốn khớp linkage còn lại (left1/left2/right1/right2) HÀN CỐ ĐỊNH ở pose 0.
+      => KHÔNG dùng <mimic> nữa: tránh lỗi "physics does not support mimic constraints"
+         và tránh các khớp tự do bị xoay lung tung khi cánh tay chuyển động.
+    - Collision là box primitive (nhẹ physics). grasp_center = điểm gắp (attach + MoveIt EE).
   -->
   <xacro:property name="gmesh" value="package://mycobot_description/meshes/adaptive_gripper"/>
   <xacro:property name="gvel" value="2.0"/>
   <xacro:property name="geff" value="20.0"/>
+  <!-- Ngón KHÔNG có collision: tránh 2 ngón tự va/kẹt cứng làm kẹt controller.
+       Việc gắp vật xử lý bằng attach/detach nên ngón không cần collision vật lý. -->
   <xacro:macro name="finger_link" params="name mesh_file ox oy oz">
     <link name="${name}">
@@ -21,8 +22,4 @@
         <origin xyz="${ox} ${oy} ${oz}" rpy="0 0 0"/>
       </visual>
-      <collision>
-        <geometry><box size="0.02 0.03 0.01"/></geometry>
-        <origin xyz="${ox} ${oy} ${oz}" rpy="0 0 0"/>
-      </collision>
       <xacro:box_inertial mass="0.02" size="0.015"/>
     </link>
@@ -45,11 +42,12 @@
     <xacro:box_inertial mass="0.1" size="0.03"/>
   </link>
+  <!-- left2/right2 (tấm bản giữa của cơ cấu 4-thanh) bị bỏ: chúng cần mimic để chuyển
+       động, mà Gazebo không hỗ trợ; giữ lại thì đứng yên và chồng lên vùng ngón đóng.
+       Giữ mỗi bên 2 link: proximal (left3/right3, được điều khiển) + tip (left1/right1). -->
   <xacro:finger_link name="gripper_left1"  mesh_file="gripper_left1.dae"  ox="0.039"  oy="-0.0133" oz="-0.012"/>
-  <xacro:finger_link name="gripper_left2"  mesh_file="gripper_left2.dae"  ox="0.005"  oy="-0.0195" oz="-0.012"/>
   <xacro:finger_link name="gripper_left3"  mesh_file="gripper_left3.dae"  ox="0.012"  oy="0.0025"  oz="-0.012"/>
   <xacro:finger_link name="gripper_right1" mesh_file="gripper_right1.dae" ox="-0.039" oy="-0.0133" oz="-0.012"/>
-  <xacro:finger_link name="gripper_right2" mesh_file="gripper_right2.dae" ox="-0.005" oy="-0.0195" oz="-0.012"/>
   <xacro:finger_link name="gripper_right3" mesh_file="gripper_right3.dae" ox="-0.012" oy="0.0025"  oz="-0.012"/>
-  <!-- Khớp điều khiển chính (đã đổi tên) -->
+  <!-- ===== 2 khớp ngón được điều khiển (đối xứng) ===== -->
   <joint name="gripper_finger_joint" type="revolute">
     <axis xyz="0 0 1"/>
@@ -59,45 +57,23 @@
     <origin xyz="-0.012 0.005 0" rpy="0 0 0"/>
   </joint>
-  <joint name="gripper_base_to_gripper_left2" type="revolute">
+  <joint name="gripper_right_joint" type="revolute">
     <axis xyz="0 0 1"/>
-    <limit effort="${geff}" lower="-0.8" upper="0.5" velocity="${gvel}"/>
+    <limit effort="${geff}" lower="-0.15" upper="0.74" velocity="${gvel}"/>
     <parent link="gripper_base"/>
-    <child link="gripper_left2"/>
-    <origin xyz="-0.005 0.027 0" rpy="0 0 0"/>
-    <mimic joint="gripper_finger_joint" multiplier="1.0" offset="0"/>
+    <child link="gripper_right3"/>
+    <origin xyz="0.012 0.005 0" rpy="0 0 0"/>
   </joint>
-  <joint name="gripper_left3_to_gripper_left1" type="revolute">
-    <axis xyz="0 0 1"/>
-    <limit effort="${geff}" lower="-0.5" upper="0.5" velocity="${gvel}"/>
+  <!-- ===== 4 khớp linkage: HÀN CỐ ĐỊNH ===== -->
+  <joint name="gripper_left3_to_gripper_left1" type="fixed">
     <parent link="gripper_left3"/>
     <child link="gripper_left1"/>
     <origin xyz="-0.027 0.016 0" rpy="0 0 0"/>
-    <mimic joint="gripper_finger_joint" multiplier="-1.0" offset="0"/>
   </joint>
-  <joint name="gripper_base_to_gripper_right3" type="revolute">
-    <axis xyz="0 0 1"/>
-    <limit effort="${geff}" lower="-0.15" upper="0.7" velocity="${gvel}"/>
-    <parent link="gripper_base"/>
-    <child link="gripper_right3"/>
-    <origin xyz="0.012 0.005 0" rpy="0 0 0"/>
-    <mimic joint="gripper_finger_joint" multiplier="-1.0" offset="0"/>
-  </joint>
-  <joint name="gripper_base_to_gripper_right2" type="revolute">
-    <axis xyz="0 0 1"/>
-    <limit effort="${geff}" lower="-0.5" upper="0.8" velocity="${gvel}"/>
-    <parent link="gripper_base"/>
-    <child link="gripper_right2"/>
-    <origin xyz="0.005 0.027 0" rpy="0 0 0"/>
-    <mimic joint="gripper_finger_joint" multiplier="-1.0" offset="0"/>
-  </joint>
-  <joint name="gripper_right3_to_gripper_right1" type="revolute">
-    <axis xyz="0 0 1"/>
-    <limit effort="${geff}" lower="-0.5" upper="0.5" velocity="${gvel}"/>
+  <joint name="gripper_right3_to_gripper_right1" type="fixed">
     <parent link="gripper_right3"/>
     <child link="gripper_right1"/>
     <origin xyz="0.027 0.016 0" rpy="0 0 0"/>
-    <mimic joint="gripper_finger_joint" multiplier="1.0" offset="0"/>
   </joint>
-  <!-- Điểm gắp: giữa 2 ngón, dùng cho attach vật + MoveIt EE. Offset tạm, tinh chỉnh Phase 6/7. -->
+  <!-- Điểm gắp: giữa 2 ngón. Offset tạm, tinh chỉnh Phase 6/7. -->
   <link name="grasp_center"/>
   <joint name="gripper_base_to_grasp_center" type="fixed">
